Commit message: tweaked robot urdf

File: turtlebot_description/urdf/turtlebot.urdf.xacro (robot description, xacro)
@@ -16,5 +16,5 @@
   <!-- Kinect sensor -->
   <xacro:property name="kinect_x_offset" value="0.176"/>    <!-- forward from base centre -->
-  <xacro:property name="kinect_z_offset" value="0.176"/>    <!-- height above top plate -->
+  <xacro:property name="kinect_z_offset" value="0.0"/>    <!-- height above top plate -->
   <!-- ======================== MATERIALS ======================== -->
   <material name="wood">

Commit message: Added bringup package to allow the encoder ticks to affect the visualization

File: turtlebot_description/urdf/turtlebot.urdf.xacro (robot description, xacro)
@@ -166,3 +166,10 @@
     <origin xyz="0 0 0" rpy="${-pi/2} 0 ${-pi/2}"/>
   </joint>
+  <!-- Alias for the frame_id published by the Kinect driver / depthimage_to_laserscan -->
+  <link name="camera_depth_frame"/>
+  <joint name="camera_depth_frame_joint" type="fixed">
+    <parent link="kinect_depth_frame"/>
+    <child link="camera_depth_frame"/>
+    <origin xyz="0 0 0" rpy="0 0 0"/>
+  </joint>
 </robot>

Commit message: Added bringup package to allow the encoder ticks to affect the visualization

File: turtlebot_description/urdf/turtlebot.urdf.xacro (robot description, xacro)
@@ -169,5 +169,5 @@
   <link name="camera_depth_frame"/>
   <joint name="camera_depth_frame_joint" type="fixed">
-    <parent link="kinect_depth_frame"/>
+    <parent link="kinect_link"/>
     <child link="camera_depth_frame"/>
     <origin xyz="0 0 0" rpy="0 0 0"/>
